File: Projects/Batboard rev 2.2/Batboard rev 2.2 w pico/Batboard rev 2.2.sch (EAGLE design)
At the start: 63 parts, among them J1 1X2-3.5MM, J2 1X2-3.5MM, J3 1X2-3.5MM, J4 1X2-3.5MM, J5 1X2-3.5MM, J6 1X2-3.5MM, U2 TL3472CD, X1 22-23-2081, X17 22-23-2081, X2 CON-MOLEX_5566-20

Commit message: Updated LEDS
Parts:
- removed C1: 100uF, SparkFun-Capacitors:100UF-POLAR-25V-20%(ELEC)
- removed C16: .47uF, SparkFun-Capacitors:1.0UF-1206-50V-10%
- removed C17: 2.2uF, SparkFun-Capacitors:1.0UF-1206-50V-10%
- removed C18: 47pF, SparkFun-Capacitors:1.0UF-1206-50V-10%
- removed C2, C6: 2uF, SparkFun-Capacitors:1.0UF-1206-50V-10%
- removed C20, C3: 10uF, SparkFun-Capacitors:1.0UF-1206-50V-10%
- removed C21: 100uF, SparkFun-Capacitors:1.0UF-1206-50V-10%
- removed C4: 0.1uF, SparkFun-Capacitors:1.0UF-1206-50V-10%
- removed C5: 4.4uF, SparkFun-Capacitors:1.0UF-1206-50V-10%
- removed C9: 13.9uF, SparkFun-Capacitors:1.0UF-1206-50V-10%
- removed R12: 22.1K, adafruit:R-US_M1206
- removed R3: 143K, adafruit:R-US_M1206
- removed R5: 10.2K, adafruit:R-US_M1206
- removed R6: 162K, adafruit:R-US_M1206
- removed R7: 10.5K, adafruit:R-US_M1206
- removed R9: 88.7K, adafruit:R-US_M1206
- removed SHOTTKY1: (no value), diode:DIODE-DO214AC
- removed SLF1: 10uH, Inductors:SLF10165
- removed SRR1260-100M1: 10uH, Inductors:SRR1260-100M
- removed TPS1: TPS54560(8), SOIC127P600X175-8N:TPS54560(8)
- removed U$5: LT1054, texas-custom:LT1054
- removed U$7: LM23630, SOIC127P602X168-8N:LM23630
Connections:
- removed net BATT: C20.1, C5.1, TPS1.VIN, U$7.EN, U$7.VIN
- removed net N$31: U$5.GND
- removed net N$46: C3.1, U$5.CAP+
- removed net N$47: C3.2, U$5.CAP-
- removed net N$52: C16.2, U$7.BOOT
- removed net N$53: C16.1, SLF1.P$1, U$7.SW
- removed net N$54: C18.1, R12.2, R9.1, U$7.FB
- removed net N$55: C17.2, U$7.VCC
- removed net N$57: C4.2, TPS1.BOOT
- removed net N$58: C4.1, SHOTTKY1.C, SRR1260-100M1.P$1, TPS1.SW
- removed net N$61: R3.1, R5.2, TPS1.FB
- removed net N$62: R6.1, TPS1.RT
- removed net N$63: R7.2, TPS1.COMP
- removed net N$64: C6.2, R7.1
- net +12V: no longer C9.1, R3.2, SRR1260-100M1.P$2
- net +5V: no longer C18.2, C21.2, R9.2, SLF1.P$2
- net -12V: no longer C1.+, C2.2, U$5.VCC, U$5.VOUT
- net GND: no longer C1.-, C17.1, C2.1, C20.2, C21.1, C5.2, C6.1, C9.2, R12.1, R5.1, R6.2, SHOTTKY1.A, U$7.AGND, U$7.PGND
Other:
- note removed: "LM23630"
