File: Projects/Batboard rev 2.2/Batboard rev 2.2 wo pico/Batboard rev 2.2.sch (EAGLE design)
At the start: 63 parts, among them J1 1X2-3.5MM, J2 1X2-3.5MM, J3 1X2-3.5MM, J4 1X2-3.5MM, J5 1X2-3.5MM, J6 1X2-3.5MM, U2 TL3472CD, X1 22-23-2081, X17 22-23-2081

Commit message: Updated LEDS
Parts:
- removed SV1: (no value), con-lstb:MA03-1
- added LED1, LED2, LED3: (no value), eagle-ltspice:LED_E
- added R1, R11, R4: 500, resistor:R-US_R1206
- added R13, R14, R15: 1K, resistor:R-US_R1206
- added U$9: DMN2004DMK_DUAL_N-CHANNEL_MOSFET_ARRAY, ultravolt_daughterboard:DMN2004DMK_DUAL_N-CHANNEL_MOSFET_ARRAY
- R2: value (none) -> 50K
Connections:
- new net 5V: R1.2, R11.2, R4.2
- new net N$31: LED1.A, R1.1
- new net N$84: LED2.A, R4.1
- new net N$85: LED3.A, R11.1
- new net N$86: LED3.C, U$9.D
- new net N$87: LED1.C, U$8.D
- new net N$88: LED2.C, U$8.D1
- net +12V: now also R13.2, U$8.G
- net +5V: now also R14.2, U$8.G1
- net -12V: now also R15.1, U$9.S
- net GND: now also R13.1, R14.1, R15.2, U$8.S, U$8.S1, U$9.G
Other:
- moved on the sheet: U2
