File: Projects/Batboard rev 2.2/Batboard rev 2.2 wo pico/Batboard rev 2.2.sch (EAGLE design)
At the start: 72 parts, among them J1 1X2-3.5MM, J2 1X2-3.5MM, J3 1X2-3.5MM, J4 1X2-3.5MM, J5 1X2-3.5MM, J6 1X2-3.5MM, U2 TL3472CD, X1 22-23-2081, X17 22-23-2081

Commit message: Update with Microphones
Parts:
- removed J4: 1X2-3.5MM, adafruit:1X2-3.5MM
- removed S1: 22-23-2021, con-molex:22-23-2021
- removed SLF1: 10uH, Inductors:SLF10165
- added SRR1260-100M2: 10uH, Inductors:SRR1260-100M
Connections:
- net +12V: no longer J4.1
- net +5V: now also SRR1260-100M2.P$2; no longer SLF1.P$2
- net -12V: now also C1.-; no longer C1.+
- net GND: now also C1.+, TPS1.GND; no longer C1.-, J4.2, S1-2.S
- net N$22: no longer S1-1.S
- net N$53: now also SRR1260-100M2.P$1; no longer SLF1.P$1
Other:
- moved on the sheet: C1
Changed lines of the file:
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@@
 <?xml version="1.0" encoding="utf-8"?>
 <!DOCTYPE eagle SYSTEM "eagle.dtd">
-<eagle version="9.0.1">
+<eagle version="9.1.1">
 <drawing>
 <settings>
@@
 <part name="GND10" library="supply1" library_urn="urn:adsk.eagle:library:371" deviceset="GND" device=""/>
 <part name="P+1" library="supply1" library_urn="urn:adsk.eagle:library:371" deviceset="+12V" device=""/>
-<part name="J4" library="adafruit" deviceset="1X2" device="-3.5MM"/>
-<part name="GND13" library="supply1" library_urn="urn:adsk.eagle:library:371" deviceset="GND" device=""/>
-<part name="P+14" library="supply1" library_urn="urn:adsk.eagle:library:371" deviceset="+12V" device=""/>
 <part name="J6" library="adafruit" deviceset="1X2" device="-3.5MM"/>
 <part name="GND15" library="supply1" library_urn="urn:adsk.eagle:library:371" deviceset="GND" device=""/>
@@
 <part name="R2" library="pot" library_urn="urn:adsk.eagle:library:331" deviceset="3RP/1610N" device="" package3d_urn="urn:adsk.eagle:package:22726/1" value="50K"/>
 <part name="SUPPLY2" library="supply2" library_urn="urn:adsk.eagle:library:372" deviceset="GND" device=""/>
-<part name="S1" library="con-molex" library_urn="urn:adsk.eagle:library:165" deviceset="22-23-2021" device=""/>
-<part name="SUPPLY3" library="supply2" library_urn="urn:adsk.eagle:library:372" deviceset="GND" device=""/>
 <part name="J2" library="adafruit" deviceset="1X2" device="-3.5MM"/>
 <part name="J3" library="adafruit" deviceset="1X2" device="-3.5MM"/>
@@
 <part name="GND37" library="SparkFun-PowerSymbols" library_urn="urn:adsk.eagle:library:530" deviceset="GND" device=""/>
 <part name="GND39" library="SparkFun-PowerSymbols" library_urn="urn:adsk.eagle:library:530" deviceset="GND" device=""/>
-<part name="C1" library="SparkFun-Capacitors" library_urn="urn:adsk.eagle:library:510" deviceset="100UF-POLAR" device="-25V-20%(ELEC)" package3d_urn="urn:adsk.eagle:package:37420/1" value="100uF"/>
 <part name="U$5" library="texas-custom" deviceset="LT1054" device=""/>
 <part name="GND9" library="SparkFun-PowerSymbols" library_urn="urn:adsk.eagle:library:530" deviceset="GND" device=""/>
@@
 </part>
 <part name="GND23" library="SparkFun-PowerSymbols" library_urn="urn:adsk.eagle:library:530" deviceset="GND" device=""/>
-<part name="SLF1" library="Inductors" deviceset="SLF10165" device="" value="10uH"/>
 <part name="C18" library="SparkFun-Capacitors" library_urn="urn:adsk.eagle:library:510" deviceset="1.0UF" device="-1206-50V-10%" package3d_urn="urn:adsk.eagle:package:37426/1" value="47pF">
 <attribute name="MF" value="KEMET"/>
@@
 <part name="GND20" library="supply1" library_urn="urn:adsk.eagle:library:371" deviceset="GND" device=""/>
 <part name="P-3" library="supply1" library_urn="urn:adsk.eagle:library:371" deviceset="-12V" device=""/>
+<part name="SRR1260-100M2" library="Inductors" deviceset="SRR1260-100M" device="" value="10uH"/>
+<part name="C1" library="SparkFun-Capacitors" library_urn="urn:adsk.eagle:library:510" deviceset="100UF-POLAR" device="-25V-20%(ELEC)" package3d_urn="urn:adsk.eagle:package:37420/1" value="100uF"/>
+<part name="GND13" library="SparkFun-PowerSymbols" library_urn="urn:adsk.eagle:library:530" deviceset="GND" device=""/>
 </parts>
 <sheets>
@@
 <attribute name="VALUE" x="-29.21" y="3.175" size="1.778" layer="96"/>
 </instance>
-<instance part="J4" gate="G$1" x="-13.97" y="1.27" smashed="yes" rot="MR0"/>
-<instance part="GND13" gate="1" x="-6.35" y="1.27" smashed="yes" rot="R90">
-<attribute name="VALUE" x="-5.715" y="0.635" size="1.778" layer="96"/>
-</instance>
-<instance part="P+14" gate="1" x="-3.81" y="3.81" smashed="yes" rot="R270">
-<attribute name="VALUE" x="-1.27" y="3.175" size="1.778" layer="96"/>
-</instance>
 <instance part="J6" gate="G$1" x="-41.91" y="-8.89" smashed="yes" rot="MR0"/>
 <instance part="GND15" gate="1" x="-34.29" y="-8.89" smashed="yes" rot="R90">
@@
 </segment>
 <segment>
-<pinref part="GND13" gate="1" pin="GND"/>
-<pinref part="J4" gate="G$1" pin="2"/>
-</segment>
-<segment>
 <pinref part="GND15" gate="1" pin="GND"/>
 <pinref part="J6" gate="G$1" pin="2"/>
@@
 <pinref part="P+1" gate="1" pin="+12V"/>
 <wire x1="-34.29" y1="3.81" x2="-36.83" y2="3.81" width="0.1524" layer="91"/>
-</segment>
-<segment>
-<pinref part="J4" gate="G$1" pin="1"/>
-<pinref part="P+14" gate="1" pin="+12V"/>
-<wire x1="-6.35" y1="3.81" x2="-8.89" y2="3.81" width="0.1524" layer="91"/>
 </segment>
 <segment>
@@
 </plain>
 <instances>
-<instance part="C1" gate="G$1" x="24.13" y="10.16"/>
 <instance part="U$5" gate="G$1" x="0" y="0"/>
 <instance part="GND9" gate="1" x="-17.78" y="-20.32" smashed="yes">
@@
 <attribute name="VALUE" x="-36.83" y="12.7" size="1.778" layer="96" rot="R180"/>
 </instance>
+<instance part="C1" gate="G$1" x="24.13" y="7.62" rot="R180"/>
 </instances>
 <busses>
@@
 <net name="GND" class="0">
 <segment>
-<pinref part="C1" gate="G$1" pin="-"/>
 <pinref part="GND11" gate="1" pin="GND"/>
 <wire x1="24.13" y1="3.81" x2="24.13" y2="5.08" width="0.1524" layer="91"/>
+<pinref part="C1" gate="G$1" pin="+"/>
 </segment>
 <segment>
@@
 <segment>
 <pinref part="U$5" gate="G$1" pin="VOUT"/>
-<pinref part="C1" gate="G$1" pin="+"/>
 <wire x1="24.13" y1="12.7" x2="15.24" y2="12.7" width="0.1524" layer="91"/>
 <wire x1="24.13" y1="12.7" x2="33.02" y2="12.7" width="0.1524" layer="91"/>
+<label x="34.29" y="12.7" size="1.778" layer="95"/>
+<pinref part="C1" gate="G$1" pin="-"/>
 <junction x="24.13" y="12.7"/>
-<label x="34.29" y="12.7" size="1.778" layer="95"/>
 </segment>
 </net>
@@
 <instance part="GND39" gate="1" x="-38.1" y="26.67" rot="R270"/>
 <instance part="C9" gate="G$1" x="39.37" y="46.99"/>
+<instance part="GND13" gate="1" x="10.16" y="34.29" rot="R90"/>
 </instances>
 <busses>
@@
 <pinref part="GND39" gate="1" pin="GND"/>
 <wire x1="-35.56" y1="26.67" x2="-31.75" y2="26.67" width="0.1524" layer="91"/>
+</segment>
+<segment>
+<pinref part="GND13" gate="1" pin="GND"/>
+<pinref part="TPS1" gate="G$1" pin="GND"/>
+<wire x1="7.62" y1="34.29" x2="5.08" y2="34.29" width="0.1524" layer="91"/>
 </segment>
 </net>
@@
 <attribute name="VALUE" x="-23.114" y="-2.54" size="1.778" layer="96" rot="R270" align="top-center"/>
 </instance>
-<instance part="SLF1" gate="G$1" x="2.54" y="13.97" smashed="yes">
-<attribute name="VALUE" x="-2.54" y="16.51" size="1.778" layer="96"/>
-<attribute name="NAME" x="3.81" y="16.51" size="1.778" layer="95"/>
-</instance>
 <instance part="C18" gate="G$1" x="17.78" y="16.51" smashed="yes">
 <attribute name="OC_FARNELL" x="17.78" y="16.51" size="1.778" layer="96" rot="R270" display="off"/>
@@
 </instance>
 <instance part="C15" gate="G$1" x="38.1" y="19.05" rot="R180"/>
+<instance part="SRR1260-100M2" gate="G$1" x="2.54" y="13.97"/>
 </instances>
 <busses>
@@
 <net name="+5V" class="0">
 <segment>
-<pinref part="SLF1" gate="G$1" pin="P$2"/>
 <wire x1="10.16" y1="13.97" x2="17.78" y2="13.97" width="0.1524" layer="91"/>
 <wire x1="17.78" y1="13.97" x2="25.4" y2="13.97" width="0.1524" layer="91"/>
@@
 <junction x="38.1" y="13.97"/>
 <pinref part="C15" gate="G$1" pin="+"/>
+<pinref part="SRR1260-100M2" gate="G$1" pin="P$2"/>
 </segment>
 </net>
@@
 <wire x1="-22.86" y1="2.54" x2="-22.86" y2="7.62" width="0.1524" layer="91"/>
 <wire x1="-22.86" y1="7.62" x2="-10.16" y2="7.62" width="0.1524" layer="91"/>
-<pinref part="SLF1" gate="G$1" pin="P$1"/>
 <wire x1="-22.86" y1="7.62" x2="-22.86" y2="13.97" width="0.1524" layer="91"/>
 <wire x1="-22.86" y1="13.97" x2="-5.08" y2="13.97" width="0.1524" layer="91"/>
 <junction x="-22.86" y="7.62"/>
+<pinref part="SRR1260-100M2" gate="G$1" pin="P$1"/>
 </segment>
 </net>
@@
 <attribute name="VALUE" x="76.835" y="-5.715" size="1.778" layer="96" rot="R270"/>
 </instance>
-<instance part="S1" gate="-1" x="85.09" y="19.05" smashed="yes">
-<attribute name="NAME" x="87.63" y="18.288" size="1.524" layer="95"/>
-<attribute name="VALUE" x="84.328" y="20.447" size="1.778" layer="96"/>
-</instance>
-<instance part="S1" gate="-2" x="85.09" y="16.51" smashed="yes">
-<attribute name="NAME" x="87.63" y="15.748" size="1.524" layer="95"/>
-</instance>
-<instance part="SUPPLY3" gate="GND" x="78.74" y="16.51" smashed="yes" rot="R270">
-<attribute name="VALUE" x="75.565" y="18.415" size="1.778" layer="96" rot="R270"/>
-</instance>
 <instance part="J2" gate="G$1" x="90.17" y="2.54" smashed="yes" rot="MR180"/>
 <instance part="J3" gate="G$1" x="90.17" y="-7.62" smashed="yes" rot="MR180"/>
@@
 <wire x1="82.55" y1="-7.62" x2="85.09" y2="-7.62" width="0.1524" layer="91"/>
 <pinref part="J3" gate="G$1" pin="2"/>
-</segment>
-<segment>
-<pinref part="S1" gate="-2" pin="S"/>
-<pinref part="SUPPLY3" gate="GND" pin="GND"/>
-<wire x1="81.28" y1="16.51" x2="82.55" y2="16.51" width="0.1524" layer="91"/>
 </segment>
 <segment>
@@
 <wire x1="72.39" y1="0" x2="72.39" y2="-10.16" width="0.1524" layer="91"/>
 <wire x1="72.39" y1="-10.16" x2="85.09" y2="-10.16" width="0.1524" layer="91"/>
-<wire x1="82.55" y1="19.05" x2="72.39" y2="19.05" width="0.1524" layer="91"/>
-<pinref part="S1" gate="-1" pin="S"/>
-<wire x1="72.39" y1="10.16" x2="72.39" y2="19.05" width="0.1524" layer="91"/>
 <pinref part="R21" gate="G$1" pin="1"/>
 <wire x1="40.64" y1="16.51" x2="59.69" y2="16.51" width="0.1524" layer="91"/>

Commit message: Havent done this in a while
Parts:
- TPS1: value TPS54560(8) -> TPS54560
Other:
- note added: "TPS54560"
Changed lines of the file:
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@@
 <?xml version="1.0" encoding="utf-8"?>
 <!DOCTYPE eagle SYSTEM "eagle.dtd">
-<eagle version="9.1.1">
+<eagle version="9.1.3">
 <drawing>
 <settings>
@@
 <part name="GND14" library="SparkFun-PowerSymbols" library_urn="urn:adsk.eagle:library:530" deviceset="GND" device=""/>
 <part name="P+5" library="supply1" library_urn="urn:adsk.eagle:library:371" deviceset="+12V" device=""/>
-<part name="TPS1" library="SOIC127P600X175-8N" deviceset="TPS54560(8)" device=""/>
+<part name="TPS1" library="SOIC127P600X175-8N" deviceset="TPS54560(8)" device="" value="TPS54560"/>
 <part name="C4" library="SparkFun-Capacitors" library_urn="urn:adsk.eagle:library:510" deviceset="1.0UF" device="-1206-50V-10%" package3d_urn="urn:adsk.eagle:package:37426/1" value="0.1uF">
 <attribute name="MF" value="KEMET"/>
@@
 <sheet>
 <plain>
+<text x="-11.43" y="13.97" size="1.778" layer="91">TPS54560</text>
 </plain>
 <instances>
